File: hardware_buck/hardware_buck.kicad_sch (KiCad schematic)
At the start: 26 parts, among them IC1 TPS40305DRCT, J1 Screw_Terminal_01x02, Q1 NTMFS5C628NLT1G, Q2 NTMFS5C628NLT1G

Commit message: schematic complete
Parts:
- added C13: 47u, symbol Device:C
- added C14: 10u, symbol Device:C
- added C15: 100n, symbol Device:C
- added J2: Screw_Terminal_01x02, symbol Connector:Screw_Terminal_01x02
- added R10, R9: 1m, symbol Device:R
Connections:
- net GND: now also C13.2, C14.2, C15.2, J2.1 (Pin_1)
- net VCC: now also C13.1, C14.1, C15.1, R9.2; no longer J1.2 (Pin_2)
- net VOUT: now also R10.2
- new net: J1.2 (Pin_2), R9.1
- new net: J2.2 (Pin_2), R10.1

Commit message: schematic complete
Parts:
- removed J1, J2: Screw_Terminal_01x02, symbol Connector:Screw_Terminal_01x02
- added C16, C17, C18, C19, C20, C21, C22, C23, C24, C25: 22u, Capacitor_SMD:C_0805_2012Metric, symbol Device:C
- added H1, H2, H3, H4: MountingHole_Pad, MountingHole:MountingHole_2.5mm_Pad_Via, symbol Mechanical:MountingHole_Pad
- added H10, H5, H6, H7, H8, H9: MountingHole, MountingHole:MountingHole_2.5mm, symbol Mechanical:MountingHole
- added TP2, TP3, TP4, TP5: TestPoint, TestPoint:TestPoint_Pad_D2.0mm, symbol Connector:TestPoint
- C1: value 100u -> 22u; footprint (none) -> Capacitor_SMD:C_0805_2012Metric
- C11, C15, C4, C6: footprint (none) -> Capacitor_SMD:C_0402_1005Metric
- C13, C2: value 47u -> 22u; footprint (none) -> Capacitor_SMD:C_0805_2012Metric
- C14, C3: footprint (none) -> Capacitor_SMD:C_0603_1608Metric
- R1, R6: footprint (none) -> Resistor_SMD:R_0402_1005Metric
- R10, R9: footprint (none) -> Resistor_SMD:R_1206_3216Metric
- TP1: footprint (none) -> TestPoint:TestPoint_Pad_D1.0mm
Connections:
- net GND: now also C16.2, C17.2, C18.2, C19.2, C20.2, C21.2, C22.2, C23.2, C24.2, C25.2, H2.1, H4.1
- net VCC: now also C23.1, C24.1, C25.1, TP3.1; no longer C13.1
- net VOUT: now also C13.1, C16.1, C17.1, C18.1, C19.1, C20.1, C21.1, C22.1, TP5.1
- net at R9.1: now also H1.1, TP2.1
- net at R10.1: now also H3.1, TP4.1
Other:
- note added: "Connect GNDS to GND Via a 0.2mm thick trace."
- moved on the sheet: C10, C11, C12, C14, C15, C3, C4, C5, C6, C7, C8, C9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

Commit message: started with the PCB layout
Parts:
- removed H10, H9: MountingHole, MountingHole:MountingHole_2.5mm, symbol Mechanical:MountingHole
- H5, H6, H7, H8: footprint MountingHole:MountingHole_2.5mm -> MountingHole:MountingHole_2.1mm
- L1: footprint (none) -> Inductor_SMD:L_7.3x7.3_H4.5
- Q1, Q2: footprint imported:TRANS_AONR21307 -> imported:NTMFS5C460NLT1G
Connections:
- net SW: now also Q2.5 (D), Q2.6 (D), Q2.7 (D), Q2.8 (D), Q2.9 (D); no longer Q2.5_6_7_8 (D)
- net VCC: now also Q1.5 (D), Q1.6 (D), Q1.7 (D), Q1.8 (D), Q1.9 (D); no longer Q1.5_6_7_8 (D)
Changed lines of the file:
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@@
 			)
 		)
-		(property "Footprint" ""
+		(property "Footprint" "Inductor_SMD:L_7.3x7.3_H4.5"
 			(at 209.55 83.82 0)
 			(effects
@@
 			)
 		)
-		(property "Footprint" "MountingHole:MountingHole_2.5mm"
+		(property "Footprint" "MountingHole:MountingHole_2.1mm"
 			(at 199.39 157.48 0)
 			(effects
@@
 	)
 	(symbol
+		(lib_name "NMOS_1")
 		(lib_id "Simulation_SPICE:NMOS")
 		(at 182.88 92.71 0)
@@
 			)
 		)
-		(property "Footprint" "imported:TRANS_AONR21307"
+		(property "Footprint" "imported:NTMFS5C460NLT1G"
 			(at 187.96 90.17 0)
 			(effects
@@
 		(pin "4"
 		)
-		(pin "5_6_7_8"
+		(pin "6"
 		)
 		(pin "3"
@@
 		(pin "1"
 		)
+		(pin "5"
+		)
+		(pin "9"
+		)
+		(pin "7"
+		)
+		(pin "8"
+		)
 		(instances
 			(project "hardware_buck"
@@
 	)
 	(symbol
-		(lib_id "Mechanical:MountingHole")
-		(at 241.3 151.13 0)
-		(unit 1)
-		(exclude_from_sim no)
-		(in_bom no)
-		(on_board yes)
-		(dnp no)
-		(fields_autoplaced yes)
-		(property "Reference" "H9"
-			(at 243.84 149.8599 0)
-			(effects
-				(font
-					(size 1.27 1.27)
-				)
-				(justify left)
-			)
-		)
-		(property "Value" "MountingHole"
-			(at 243.84 152.3999 0)
-			(effects
-				(font
-					(size 1.27 1.27)
-				)
-				(justify left)
-			)
-		)
-		(property "Footprint" "MountingHole:MountingHole_2.5mm"
-			(at 241.3 151.13 0)
-			(effects
-				(font
-					(size 1.27 1.27)
-				)
-				(hide yes)
-			)
-		)
-		(property "Datasheet" "~"
-			(at 241.3 151.13 0)
-			(effects
-				(font
-					(size 1.27 1.27)
-				)
-				(hide yes)
-			)
-		)
-		(property "Description" "Mounting Hole without connection"
-			(at 241.3 151.13 0)
-			(effects
-				(font
-					(size 1.27 1.27)
-				)
-				(hide yes)
-			)
-		)
-		(instances
-			(project ""
-				(path "/c1ad8cd5-e773-4e08-986d-f57eb33e4793"
-					(reference "H9")
-					(unit 1)
-				)
-			)
-		)
-	)
-	(symbol
 		(lib_id "Device:C")
 		(at 69.85 130.81 0)
@@
 	)
 	(symbol
-		(lib_id "Mechanical:MountingHole")
-		(at 241.3 157.48 0)
-		(unit 1)
-		(exclude_from_sim no)
-		(in_bom no)
-		(on_board yes)
-		(dnp no)
-		(fields_autoplaced yes)
-		(property "Reference" "H10"
-			(at 243.84 156.2099 0)
-			(effects
-				(font
-					(size 1.27 1.27)
-				)
-				(justify left)
-			)
-		)
-		(property "Value" "MountingHole"
-			(at 243.84 158.7499 0)
-			(effects
-				(font
-					(size 1.27 1.27)
-				)
-				(justify left)
-			)
-		)
-		(property "Footprint" "MountingHole:MountingHole_2.5mm"
-			(at 241.3 157.48 0)
-			(effects
-				(font
-					(size 1.27 1.27)
-				)
-				(hide yes)
-			)
-		)
-		(property "Datasheet" "~"
-			(at 241.3 157.48 0)
-			(effects
-				(font
-					(size 1.27 1.27)
-				)
-				(hide yes)
-			)
-		)
-		(property "Description" "Mounting Hole without connection"
-			(at 241.3 157.48 0)
-			(effects
-				(font
-					(size 1.27 1.27)
-				)
-				(hide yes)
-			)
-		)
-		(instances
-			(project "hardware_buck"
-				(path "/c1ad8cd5-e773-4e08-986d-f57eb33e4793"
-					(reference "H10")
-					(unit 1)
-				)
-			)
-		)
-	)
-	(symbol
 		(lib_id "Device:C")
 		(at 77.47 106.68 0)
@@
 			)
 		)
-		(property "Footprint" "MountingHole:MountingHole_2.5mm"
+		(property "Footprint" "MountingHole:MountingHole_2.1mm"
 			(at 199.39 151.13 0)
 			(effects
@@
 				)
 				(justify left)
+				(hide yes)
 			)
 		)
@@
 				)
 				(justify left)
+				(hide yes)
 			)
 		)
-		(property "Footprint" "imported:TRANS_AONR21307"
+		(property "Footprint" "imported:NTMFS5C460NLT1G"
 			(at 187.96 72.39 0)
 			(effects
@@
 		(pin "4"
 		)
-		(pin "5_6_7_8"
+		(pin "7"
 		)
 		(pin "3"
@@
 		(pin "1"
 		)
+		(pin "6"
+		)
+		(pin "8"
+		)
+		(pin "9"
+		)
+		(pin "5"
+		)
 		(instances
 			(project ""
@@
 			)
 		)
-		(property "Footprint" "MountingHole:MountingHole_2.5mm"
+		(property "Footprint" "MountingHole:MountingHole_2.1mm"
 			(at 219.71 157.48 0)
 			(effects
@@
 			)
 		)
-		(property "Footprint" "MountingHole:MountingHole_2.5mm"
+		(property "Footprint" "MountingHole:MountingHole_2.1mm"
 			(at 219.71 151.13 0)
 			(effects
